Commit message: Update body_link -> base_link. Standard usage (e.g., nav2).

File: usd_assets/robot.urdf (robot description, URDF)
Before this commit: robot differential_drive_robot_4wheel, 10 links, 9 joints
Links:
- removed link body_link
- added link base_link, mass 4.6655999999999995; collision box size=0.24 0.12 0.06; visual box size=0.24 0.12 0.06
Joints:
- joint battery_joint: parent body_link -> base_link
- joint left_wheel2_joint: parent body_link -> base_link
- joint left_wheel_joint: parent body_link -> base_link
- joint right_wheel2_joint: parent body_link -> base_link
- joint right_wheel_joint: parent body_link -> base_link
